File: FlightComputer/ESP32-FC/ESP32-FC/ESP32-FC.kicad_pcb (KiCad board)
At the start: 2 copper layers, 55 x 40 mm, 19 parts, among them J1 USB_C_Receptacle_USB2.0_16P, U1 ESP32-S3-WROOM-1, U2 AP2112K-3.3, U3 ICP-20100, U4 ICM-42670-P

Commit message: Part placement
Parts:
- added C10: C, Capacitor_SMD:C_0201_0603Metric_Pad0.64x0.40mm_HandSolder, F.Cu at (150.0, 91.7)
- added C11: C, Capacitor_SMD:C_0201_0603Metric_Pad0.64x0.40mm_HandSolder, F.Cu at (154.7, 93.0)
- added C8: C, Capacitor_SMD:C_0201_0603Metric_Pad0.64x0.40mm_HandSolder, F.Cu at (146.3, 85.3)
- added C9: C, Capacitor_SMD:C_0201_0603Metric_Pad0.64x0.40mm_HandSolder, F.Cu at (146.2, 87.6)
- added D1: D_Schottky, Diode_SMD:D_0201_0603Metric_Pad0.64x0.40mm_HandSolder, F.Cu at (150.7, 87.9)
- added D2: D_Schottky, Diode_SMD:D_0201_0603Metric_Pad0.64x0.40mm_HandSolder, F.Cu at (150.5, 90.8)
- added D3: D_Schottky, Diode_SMD:D_0201_0603Metric_Pad0.64x0.40mm_HandSolder, F.Cu at (154.5, 88.3)
- added D4: LED, LED_SMD:LED_0201_0603Metric_Pad0.64x0.40mm_HandSolder, F.Cu at (155.5, 90.8)
- added D5: LED, LED_SMD:LED_0201_0603Metric_Pad0.64x0.40mm_HandSolder, F.Cu at (148.0, 90.1)
- added D6: LED, LED_SMD:LED_0201_0603Metric_Pad0.64x0.40mm_HandSolder, F.Cu at (147.9, 93.9)
- added D7: LED, LED_SMD:LED_0201_0603Metric_Pad0.64x0.40mm_HandSolder, F.Cu at (156.2, 106.8)
- added H1: MountingHole, MountingHole:MountingHole_3mm, F.Cu at (173.7, 84.8)
- added H2: MountingHole, MountingHole:MountingHole_3mm, F.Cu at (173.7, 115.0)
- added H3: MountingHole, MountingHole:MountingHole_3mm, F.Cu at (127.2, 84.5)
- added H4: MountingHole, MountingHole:MountingHole_3mm, F.Cu at (126.5, 116.2)
- added J2: Conn_01x02_Pin, Connector_JST:JST_PH_B2B-PH-K_1x02_P2.00mm_Vertical, F.Cu at (142.8, 83.9)
- added J3: Conn_01x04_Pin, Connector_PinHeader_2.54mm:PinHeader_1x04_P2.54mm_Vertical, F.Cu at (158.1, 117.5)
- added J4: Conn_01x03_Pin, Connector_PinHeader_2.54mm:PinHeader_1x03_P2.54mm_Vertical, F.Cu at (141.4, 91.8)
- added J5: Conn_01x03_Pin, Connector_PinHeader_2.54mm:PinHeader_1x03_P2.54mm_Vertical, F.Cu at (141.4, 102.0)
- added L1: L, Inductor_SMD:L_0201_0603Metric_Pad0.64x0.40mm_HandSolder, F.Cu at (149.6, 87.0)
- added R10: R, Resistor_SMD:R_0201_0603Metric_Pad0.64x0.40mm_HandSolder, F.Cu at (146.8, 82.0)
- added R11: R, Resistor_SMD:R_0201_0603Metric_Pad0.64x0.40mm_HandSolder, F.Cu at (148.4, 95.0)
- added R12: R, Resistor_SMD:R_0201_0603Metric_Pad0.64x0.40mm_HandSolder, F.Cu at (154.4, 89.6)
- added R13: R, Resistor_SMD:R_0201_0603Metric_Pad0.64x0.40mm_HandSolder, F.Cu at (148.1, 89.1)
- added R14: R, Resistor_SMD:R_0201_0603Metric_Pad0.64x0.40mm_HandSolder, F.Cu at (147.9, 92.9)
- added R15: R, Resistor_SMD:R_0201_0603Metric_Pad0.64x0.40mm_HandSolder, F.Cu at (172.2, 89.5)
- added R8: R, Resistor_SMD:R_0201_0603Metric_Pad0.64x0.40mm_HandSolder, F.Cu at (153.4, 84.2)
- added R9: R, Resistor_SMD:R_0201_0603Metric_Pad0.64x0.40mm_HandSolder, F.Cu at (151.9, 83.4)
- added SW1: BOOT, Button_Switch_SMD:SW_Push_SPST_NO_Alps_SKRK, F.Cu at (153.3, 110.8)
- added SW2: RESET, Button_Switch_SMD:SW_Push_SPST_NO_Alps_SKRK, F.Cu at (168.6, 88.1)
- added U5: MT3608, Package_TO_SOT_SMD:SOT-23-6, F.Cu at (149.2, 84.6)
- C1, C2, C3, C4, C5, C6, C7: footprint Capacitor_SMD:C_0805_2012Metric_Pad1.18x1.45mm_HandSolder -> Capacitor_SMD:C_0201_0603Metric_Pad0.64x0.40mm_HandSolder
- R1, R2, R3, R4, R5: footprint Resistor_SMD:R_0805_2012Metric_Pad1.20x1.40mm_HandSolder -> Resistor_SMD:R_0201_0603Metric_Pad0.64x0.40mm_HandSolder
- R6, R7: value R -> 4K7; footprint Resistor_SMD:R_0805_2012Metric_Pad1.20x1.40mm_HandSolder -> Resistor_SMD:R_0201_0603Metric_Pad0.64x0.40mm_HandSolder
- moved C1 97.3 mm to (175.9, 90.8)
- moved C2 93.9 mm to (173.9, 90.7), turned to 180 degrees
- moved C3 84.5 mm to (155.2, 100.3), turned to -90 degrees
- moved C6 79.2 mm to (169.1, 83.0), turned to -90 degrees
- moved C5 78.9 mm to (153.0, 100.8)
- moved C4 78.7 mm to (154.1, 96.4)
- moved R1 78.2 mm to (154.9, 106.8), turned to 90 degrees
- moved C7 74.5 mm to (166.4, 80.9)
- moved R2 71.2 mm to (162.3, 87.6)
- moved R6 68.3 mm to (162.8, 91.1)
- moved R3 65.0 mm to (156.9, 87.6), turned to 180 degrees
- moved R7 62.8 mm to (156.2, 95.7)
- moved U3 27.8 mm to (167.3, 82.7)
- moved U4 17.2 mm to (153.0, 98.8)
- moved U2 16.0 mm to (151.6, 93.9)
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Connections:
- J1 pad A4: +5V -> Net-(D3-A)
- J1 pad A9: +5V -> Net-(D3-A)
- J1 pad B4: +5V -> Net-(D3-A)
- J1 pad B9: +5V -> Net-(D3-A)
- R1 pad 1: unconnected-(R1-Pad1) -> Net-(D7-K)
- R1 pad 2: unconnected-(R1-Pad2) -> GND
- U1 pad 10: unconnected-(U1-IO17-Pad10) -> /ESP_TX
- U1 pad 11: unconnected-(U1-IO18-Pad11) -> /ESP_RX
- U1 pad 22: unconnected-(U1-IO14-Pad22) -> /SERVO2
- U1 pad 25: unconnected-(U1-IO48-Pad25) -> Net-(D7-A)
- U1 pad 27: unconnected-(U1-IO0-Pad27) -> Net-(U1-IO0)
- U1 pad 3: unconnected-(U1-EN-Pad3) -> /EN
- U1 pad 39: unconnected-(U1-IO1-Pad39) -> /SERVO1
- U2 pad 1: unconnected-(U2-VIN-Pad1) -> +5V
- U2 pad 2: unconnected-(U2-GND-Pad2) -> GND
- U2 pad 3: unconnected-(U2-EN-Pad3) -> Net-(U2-EN)
- U2 pad 5: unconnected-(U2-VOUT-Pad5) -> +3V3

Commit message: Layout Major
Parts:
- added G***: LOGO, LOGO, F.Cu at (143.6, 103.1)
- moved H4 7.95 mm to (134.5, 116.0)
- moved H3 7.30 mm to (134.5, 84.0)
- moved J4 7.20 mm to (134.3, 93.3)
- moved J5 7.20 mm to (134.3, 103.4)
- moved R14 5.54 mm to (152.9, 90.6), turned to 180 degrees
- moved +3V 5.49 mm to (152.9, 91.6)
- moved D2 3.78 mm to (152.2, 87.4), turned to 90 degrees
- moved C4 3.73 mm to (156.2, 99.5), turned to -90 degrees
- moved D1 2.96 mm to (147.8, 87.8)
- moved BOOST 2.93 mm to (150.9, 89.5)
- moved C3 1.99 mm to (155.9, 102.2)
- moved C5 1.99 mm to (153.7, 102.6)
- moved U4 1.99 mm to (153.7, 100.7)
- moved L1 1.80 mm to (147.8, 86.9)
- moved C2 1.55 mm to (175.5, 90.9), turned to 0 degrees
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- renumbered D6 to +3V, D4 to +5V, D5 to BOOST, SW1 to BOOT, D7 to GPIO, SW2 to RESET
Routing:
- net +3V3: track 0.00 -> 92.8 mm, vias 0 -> 8
- net GND: track 0.00 -> 79.2 mm, vias 0 -> 110
- net /SERVO1: track 0.00 -> 46.9 mm, vias 0 -> 2
- net +5V: track 0.00 -> 42.1 mm
- net /SCL: track 0.00 -> 29.0 mm, vias 0 -> 3
- net /SERVO2: track 0.00 -> 26.2 mm
- net /ESP_RX: track 0.00 -> 25.9 mm, vias 0 -> 2
- net /ESP_TX: track 0.00 -> 25.4 mm, vias 0 -> 2
- net /SDA: track 0.00 -> 24.1 mm, vias 0 -> 2
- net VBAT: track 0.00 -> 12.8 mm
- net Net-(D1-A): track 0.00 -> 10.8 mm
- net Net-(D3-A): track 0.00 -> 9.78 mm
- net USB_D-: track 0.00 -> 9.17 mm
- net USB_D+: track 0.00 -> 7.98 mm
- net /EN: track 0.00 -> 7.53 mm
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- added copper zone on In1.Cu, net GND
Other:
- board size 55 x 40 mm -> 47 x 40 mm
- copper layers 2 -> 4
- board text added: "Team 'Lite Work ESP32 Board Designed By: Fawaaz Kamali Siddiqui"
